Commit message: update

File: robot_description/yuuki_biped.urdf (robot description, URDF)
Before this commit: robot yuuki_biped, 14 links, 13 joints
Links:
- link left_ankle: geometry collision box size=0.03 0.048 0.061; visual box size=0.03 0.048 0.061
- link left_hip: geometry collision box size=0.03 0.048 0.061; visual box size=0.03 0.048 0.061
- link left_shin: geometry collision box size=0.03 0.048 0.065; collision box size=0.032 0.048 0.153
- link left_thigh: geometry collision box size=0.03 0.048 0.065; collision box size=0.032 0.048 0.153
- link right_ankle: geometry collision box size=0.03 0.048 0.061; visual box size=0.03 0.048 0.061
- link right_hip: geometry collision box size=0.03 0.048 0.061; visual box size=0.03 0.048 0.061
- link right_shin: geometry collision box size=0.03 0.048 0.065; collision box size=0.032 0.048 0.153
- link right_thigh: geometry collision box size=0.03 0.048 0.065; collision box size=0.032 0.048 0.153
Joints:
- joint left_sole_fixed: origin xyz=0.05 0 -0.04 rpy=0 0 0 -> xyz=0.05 0 -0.058 rpy=0 0 0
- joint right_sole_fixed: origin xyz=0.05 0 -0.04 rpy=0 0 0 -> xyz=0.05 0 -0.058 rpy=0 0 0

Commit message: update

File: robot_description/yuuki_biped.urdf (robot description, URDF)
Before this commit: robot yuuki_biped, 14 links, 13 joints
Links:
- link left_foot: geometry collision box size=0.048 0.03 0.065; collision box size=0.3 0.17 0.002
- link left_hip: geometry collision box size=0.048 0.03 0.061; visual box size=0.048 0.03 0.061
- link right_foot: geometry collision box size=0.048 0.03 0.065; collision box size=0.3 0.17 0.002
- link right_hip: geometry collision box size=0.048 0.03 0.061; visual box size=0.048 0.03 0.061
